File: reset.kicad_sch (KiCad schematic)
At the start: 46 parts, among them J7 JST_SH_1x8_BM08B-SRSS-TB-LF-SN, Q8 DTC014T_SOT-416, Q9 DTC014T_SOT-416, U31 TPS3840PH30DBVR, U32 TPS3840PH30DBVR, U33 74AVC4T245_UQFN, U34 SN74AVC2T245_UQFN, U35 SN74LVC1G125_SOT, U36 74LCX07_QFN

Commit message: Removed camera connector from schematic and pcb
Parts:
- removed TP22: TP_0.75mm_SMD, kria-k26-devboard-footprints:TP_SMD_0.75mm, symbol kria-k26-devboard:TP_0.75mm_SMD
- C133, C135, D4, U32, U35: now not fitted
Connections:
- net CAM_RST: no longer J7.3 (Pin_3)
- no-connect marks 4 -> 5
Changed lines of the file:
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@@
 	)
 	(junction
-		(at 365.125 149.86)
-		(diameter 0)
-		(color 0 0 0 0)
-	)
-	(junction
 		(at 311.15 41.91)
 		(diameter 0)
@@
 	)
 	(no_connect
+		(at 373.38 149.86)
+	)
+	(no_connect
 		(at 303.53 125.73)
 	)
@@
 	(wire
 		(pts
-			(xy 352.425 149.86) (xy 365.125 149.86)
-		)
-		(stroke
-			(width 0)
-			(type default)
-		)
-	)
-	(wire
-		(pts
 			(xy 292.735 137.16) (xy 306.07 137.16)
 		)
@@
 	(wire
 		(pts
-			(xy 365.125 133.985) (xy 365.125 149.86)
-		)
-		(stroke
-			(width 0)
-			(type default)
-		)
-	)
-	(wire
-		(pts
 			(xy 308.61 41.91) (xy 311.15 41.91)
 		)
@@
 	(wire
 		(pts
-			(xy 365.125 149.86) (xy 373.38 149.86)
-		)
-		(stroke
-			(width 0)
-			(type default)
-		)
-	)
-	(wire
-		(pts
 			(xy 341.63 44.45) (xy 341.63 41.91)
 		)
@@
 		)
 	)
-	(hierarchical_label "CAM_RST"
-		(shape input)
-		(at 352.425 149.86 180)
-		(effects
-			(font
-				(size 1.27 1.27)
-			)
-			(justify right)
-		)
-	)
 	(hierarchical_label "~{M2_PERST}"
 		(shape input)
@@
 	(symbol
 		(lib_id "kria-k26-devboard:TP_0.75mm_SMD")
-		(at 365.125 133.985 90)
-		(unit 1)
-		(exclude_from_sim no)
-		(in_bom yes)
-		(on_board yes)
-		(dnp no)
-		(property "Reference" "TP22"
-			(at 365.125 127 0)
-			(effects
-				(font
-					(size 1.27 1.27)
-				)
-			)
-		)
-		(property "Value" "TP_0.75mm_SMD"
-			(at 367.665 133.985 0)
-			(effects
-				(font
-					(size 1.27 1.27)
-					(thickness 0.15)
-				)
-				(justify left bottom)
-				(hide yes)
-			)
-		)
-		(property "Footprint" "kria-k26-devboard-footprints:TP_SMD_0.75mm"
-			(at 360.045 128.905 0)
-			(effects
-				(font
-					(size 1.27 1.27)
-					(thickness 0.15)
-				)
-				(justify left bottom)
-				(hide yes)
-			)
-		)
-		(property "Datasheet" ""
-			(at 357.505 128.905 0)
-			(effects
-				(font
-					(size 1.27 1.27)
-					(thickness 0.15)
-				)
-				(justify left bottom)
-				(hide yes)
-			)
-		)
-		(property "Description" ""
-			(at 365.125 133.985 0)
-			(effects
-				(font
-					(size 1.27 1.27)
-				)
-			)
-		)
-		(property "MPN" ""
-			(at 380.365 116.205 0)
-			(effects
-				(font
-					(size 1.27 1.27)
-					(thickness 0.15)
-				)
-				(justify left bottom)
-				(hide yes)
-			)
-		)
-		(property "Manufacturer" ""
-			(at 382.905 116.205 0)
-			(effects
-				(font
-					(size 1.27 1.27)
-					(thickness 0.15)
-				)
-				(justify left bottom)
-				(hide yes)
-			)
-		)
-		(property "Author" "Antmicro"
-			(at 385.445 116.205 0)
-			(effects
-				(font
-					(size 1.27 1.27)
-					(thickness 0.15)
-				)
-				(justify left bottom)
-				(hide yes)
-			)
-		)
-		(property "License" "Apache-2.0"
-			(at 387.985 116.205 0)
-			(effects
-				(font
-					(size 1.27 1.27)
-					(thickness 0.15)
-				)
-				(justify left bottom)
-				(hide yes)
-			)
-		)
-		(pin "1"
-		)
-		(instances
-			(project "kria-k26-devboard"
-				(path "/c38c692d-dd84-4abf-ab35-63104b24d124/00000000-0000-0000-0000-000065aaf1bf"
-					(reference "TP22")
-					(unit 1)
-				)
-			)
-		)
-	)
-	(symbol
-		(lib_id "kria-k26-devboard:TP_0.75mm_SMD")
 		(at 367.665 133.985 90)
 		(unit 1)
@@
 		(in_bom yes)
 		(on_board yes)
-		(dnp no)
+		(dnp yes)
 		(fields_autoplaced yes)
 		(property "Reference" "U32"
@@
 		(in_bom yes)
 		(on_board yes)
-		(dnp no)
+		(dnp yes)
 		(fields_autoplaced yes)
 		(property "Reference" "C135"
@@
 		(in_bom yes)
 		(on_board yes)
-		(dnp no)
+		(dnp yes)
 		(fields_autoplaced yes)
 		(property "Reference" "C133"
@@
 		(in_bom yes)
 		(on_board yes)
-		(dnp no)
+		(dnp yes)
 		(fields_autoplaced yes)
 		(property "Reference" "D4"
@@
 		(in_bom yes)
 		(on_board yes)
-		(dnp no)
+		(dnp yes)
 		(property "Reference" "U35"
 			(at 212.09 189.865 0)
