File: CAN.kicad_sch (KiCad schematic)
At the start: 0 parts

Commit message: Added CAN transceiver to project
Parts:
- added U10: TCAN1042HVDQ1, kria-k26-devboard-footprints:D0008A_L, symbol kria-k26-devboard:TCAN1042HVDQ1
Changed lines of the file:
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@@
 	(generator_version "9.0")
 	(paper "A4")
+	(symbol
+		(lib_id "kria-k26-devboard:TCAN1042HVDQ1")
+		(at 68.58 91.44 0)
+		(unit 1)
+		(exclude_from_sim no)
+		(in_bom yes)
+		(on_board yes)
+		(dnp no)
+		(fields_autoplaced yes)
+		(property "Reference" "U10"
+			(at 68.58 71.12 0)
+			(effects
+				(font
+					(size 1.524 1.524)
+				)
+			)
+		)
+		(property "Value" "TCAN1042HVDQ1"
+			(at 68.58 73.66 0)
+			(effects
+				(font
+					(size 1.524 1.524)
+				)
+			)
+		)
+		(property "Footprint" "kria-k26-devboard-footprints:D0008A_L"
+			(at 68.58 91.44 0)
+			(effects
+				(font
+					(size 1.27 1.27)
+					(italic yes)
+				)
+				(hide yes)
+			)
+		)
+		(property "Datasheet" "https://www.ti.com/lit/gpn/tcan1042hv-q1"
+			(at 68.58 91.44 0)
+			(effects
+				(font
+					(size 1.27 1.27)
+					(italic yes)
+				)
+				(hide yes)
+			)
+		)
+		(property "Description" "Automotive Fault Protected CAN Transceiver with CAN FD"
+			(at 68.58 91.44 0)
+			(effects
+				(font
+					(size 1.27 1.27)
+				)
+				(hide yes)
+			)
+		)
+		(pin "2"
+		)
+		(pin "3"
+		)
+		(pin "6"
+		)
+		(pin "7"
+		)
+		(pin "5"
+		)
+		(pin "8"
+		)
+		(pin "4"
+		)
+		(pin "1"
+		)
+		(instances
+			(project ""
+				(path "/c38c692d-dd84-4abf-ab35-63104b24d124/822e1ac9-b545-4f5a-99c6-f4ce1e3c2f79"
+					(reference "U10")
+					(unit 1)
+				)
+			)
+		)
+	)
 )
