File: k26_som.kicad_sch (KiCad schematic)
At the start: 56 parts, among them J6 PinHeader_1x2_P2.54mm_Drill1.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, M1 XILINX-KRIA-K26, Q19 DTC014T_SOT-416, Q6 PJA3441, Q7 DTC014T_SOT-416

Commit message: Added all components and finished first attempt at schematic
Connections:
- net HPA06_CLK0_N renamed HPA_CLK0_N
- net HPA06_CLK0_P renamed HPA_CLK0_P
